Commit message: 添加 tele_center link；发给机械臂的指令改为低跟随模式以获得更平滑的运动

File: dual_rm_75/dual_rm_75_description/urdf/dual_rm_75.urdf.xacro (robot description, xacro)
@@ -60,3 +60,16 @@
         driver_namespace="/right_arm"
     />
+    <!-- Teleoperation Center -->
+    <link name="left_tele_center" />
+    <joint name="left_tele_center_joint" type="fixed">
+        <origin xyz="0.0 0.0 0.1" rpy="0.0 ${radians(-90)} ${radians(-32)}"/>
+        <parent link="left_arm_flange"/>
+        <child link="left_tele_center"/>
+    </joint>
+    <link name="right_tele_center" />
+    <joint name="right_tele_center_joint" type="fixed">
+        <origin xyz="0.0 0.0 0.1" rpy="0.0 ${radians(90)} 0.0"/>
+        <parent link="right_arm_flange"/>
+        <child link="right_tele_center"/>
+    </joint>
 </robot>
